File: main.sch (EAGLE design)
At the start: 18 parts, among them U1 433MHz, U2 ATMEGA328P-MU-QFN32

Commit message: Redesign
Parts:
- added C1: 2.2µ, resistor:C-EUC0603
- added Q1: BSS84, transistor-small-signal:BSS84
- added R7, R8: (no value), resistor:R-EU_R0603
- renumbered D1 to LED_3V3, D2 to LED_5V, D3 to LED_RX, JP1 to PPM1, JP2 to PPM2, JP3 to PPM3, JP4 to SBUS
Connections:
- removed net PPM4: SBUS.2, U2.PD1(TXD/PCINT17)
- new net !SBUS: R8.2, U2.PD1(TXD/PCINT17)
- new net N$10: Q1.G, R8.1
- new net SBUS: Q1.S, R7.1, SBUS.2
- net +3V3: now also C1.1; no longer PPM1.1, PPM2.1, PPM3.1, SBUS.1
- net +5V: now also PPM1.1, PPM2.1, PPM3.1, R7.2, SBUS.1
- net GND: now also C1.2, Q1.D, U2.PAD

Commit message: Layout cleanup
Parts:
- added SJ1: (no value), jumper:SJ2W
Connections:
- new net N$6: SBUS.1, SJ1.2
- net !SBUS: now also SJ1.3
- net +5V: now also PPM1.2, PPM2.2, PPM3.2, SBUS.2; no longer PPM1.1, PPM2.1, PPM3.1, SBUS.1
- net PPM1: now also PPM1.1; no longer PPM1.2
- net PPM2: now also PPM2.1; no longer PPM2.2
- net PPM3: now also PPM3.1; no longer PPM3.2
- net SBUS: now also SJ1.1; no longer SBUS.2
Changed lines of the file:
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@@
 <part name="GND11" library="supply1" library_urn="urn:adsk.eagle:library:371" deviceset="GND" device=""/>
 <part name="SUPPLY4" library="supply2" library_urn="urn:adsk.eagle:library:372" deviceset="+5V" device=""/>
+<part name="SJ1" library="jumper" library_urn="urn:adsk.eagle:library:252" deviceset="SJ2W" device="" package3d_urn="urn:adsk.eagle:package:15474/1"/>
 </parts>
 <sheets>
@@
 <instance part="GND11" gate="1" x="111.76" y="-38.1"/>
 <instance part="SUPPLY4" gate="+5V" x="111.76" y="0"/>
+<instance part="SJ1" gate="G$1" x="167.64" y="22.86"/>
 </instances>
 <busses>
@@
 <net name="PPM1" class="0">
 <segment>
-<pinref part="PPM1" gate="A" pin="2"/>
-<wire x1="99.06" y1="20.32" x2="91.44" y2="20.32" width="0.1524" layer="91"/>
-<wire x1="91.44" y1="20.32" x2="91.44" y2="25.4" width="0.1524" layer="91"/>
 <label x="91.44" y="25.4" size="1.778" layer="95" rot="R90" xref="yes"/>
+<pinref part="PPM1" gate="A" pin="1"/>
+<wire x1="91.44" y1="22.86" x2="91.44" y2="25.4" width="0.1524" layer="91"/>
+<wire x1="99.06" y1="22.86" x2="91.44" y2="22.86" width="0.1524" layer="91"/>
 </segment>
 <segment>
@@
 <net name="PPM2" class="0">
 <segment>
-<pinref part="PPM2" gate="A" pin="2"/>
-<wire x1="114.3" y1="20.32" x2="106.68" y2="20.32" width="0.1524" layer="91"/>
-<wire x1="106.68" y1="20.32" x2="106.68" y2="25.4" width="0.1524" layer="91"/>
 <label x="106.68" y="25.4" size="1.778" layer="95" rot="R90" xref="yes"/>
+<pinref part="PPM2" gate="A" pin="1"/>
+<wire x1="106.68" y1="22.86" x2="106.68" y2="25.4" width="0.1524" layer="91"/>
+<wire x1="114.3" y1="22.86" x2="106.68" y2="22.86" width="0.1524" layer="91"/>
 </segment>
 <segment>
@@
 <net name="PPM3" class="0">
 <segment>
-<pinref part="PPM3" gate="A" pin="2"/>
-<wire x1="129.54" y1="20.32" x2="121.92" y2="20.32" width="0.1524" layer="91"/>
-<wire x1="121.92" y1="20.32" x2="121.92" y2="25.4" width="0.1524" layer="91"/>
 <label x="121.92" y="25.4" size="1.778" layer="95" rot="R90" xref="yes"/>
+<pinref part="PPM3" gate="A" pin="1"/>
+<wire x1="121.92" y1="22.86" x2="121.92" y2="25.4" width="0.1524" layer="91"/>
+<wire x1="129.54" y1="22.86" x2="121.92" y2="22.86" width="0.1524" layer="91"/>
 </segment>
 <segment>
@@
 </segment>
 <segment>
+<label x="76.2" y="-22.86" size="1.778" layer="95" rot="R180" xref="yes"/>
 <pinref part="R8" gate="G$1" pin="2"/>
-<wire x1="93.98" y1="-22.86" x2="88.9" y2="-22.86" width="0.1524" layer="91"/>
-<label x="88.9" y="-22.86" size="1.778" layer="95" rot="R180" xref="yes"/>
+<wire x1="76.2" y1="-22.86" x2="93.98" y2="-22.86" width="0.1524" layer="91"/>
+</segment>
+<segment>
+<pinref part="SJ1" gate="G$1" pin="3"/>
+<wire x1="167.64" y1="17.78" x2="167.64" y2="12.7" width="0.1524" layer="91"/>
+<wire x1="167.64" y1="12.7" x2="162.56" y2="12.7" width="0.1524" layer="91"/>
+<label x="162.56" y="12.7" size="1.778" layer="95" rot="R180" xref="yes"/>
 </segment>
 </net>
@@
 </segment>
 <segment>
-<pinref part="PPM1" gate="A" pin="1"/>
-<pinref part="PPM2" gate="A" pin="1"/>
-<wire x1="99.06" y1="22.86" x2="114.3" y2="22.86" width="0.1524" layer="91"/>
-<pinref part="PPM3" gate="A" pin="1"/>
-<wire x1="114.3" y1="22.86" x2="129.54" y2="22.86" width="0.1524" layer="91"/>
-<junction x="114.3" y="22.86"/>
-<pinref part="SBUS" gate="A" pin="1"/>
-<wire x1="129.54" y1="22.86" x2="144.78" y2="22.86" width="0.1524" layer="91"/>
-<junction x="129.54" y="22.86"/>
-<wire x1="99.06" y1="22.86" x2="86.36" y2="22.86" width="0.1524" layer="91"/>
-<junction x="99.06" y="22.86"/>
-<wire x1="86.36" y1="22.86" x2="86.36" y2="25.4" width="0.1524" layer="91"/>
 <pinref part="SUPPLY3" gate="+5V" pin="+5V"/>
+<wire x1="86.36" y1="25.4" x2="86.36" y2="20.32" width="0.1524" layer="91"/>
+<pinref part="PPM1" gate="A" pin="2"/>
+<wire x1="86.36" y1="20.32" x2="99.06" y2="20.32" width="0.1524" layer="91"/>
+<pinref part="PPM2" gate="A" pin="2"/>
+<wire x1="99.06" y1="20.32" x2="114.3" y2="20.32" width="0.1524" layer="91"/>
+<junction x="99.06" y="20.32"/>
+<pinref part="PPM3" gate="A" pin="2"/>
+<wire x1="114.3" y1="20.32" x2="129.54" y2="20.32" width="0.1524" layer="91"/>
+<junction x="114.3" y="20.32"/>
+<pinref part="SBUS" gate="A" pin="2"/>
+<wire x1="129.54" y1="20.32" x2="144.78" y2="20.32" width="0.1524" layer="91"/>
+<junction x="129.54" y="20.32"/>
 </segment>
 <segment>
@@
 </net>
 <net name="SBUS" class="0">
-<segment>
-<pinref part="SBUS" gate="A" pin="2"/>
-<wire x1="144.78" y1="20.32" x2="137.16" y2="20.32" width="0.1524" layer="91"/>
-<wire x1="137.16" y1="20.32" x2="137.16" y2="25.4" width="0.1524" layer="91"/>
-<label x="137.16" y="25.4" size="1.778" layer="95" rot="R90" xref="yes"/>
-</segment>
 <segment>
 <pinref part="Q1" gate="G$1" pin="S"/>
@@
 <label x="127" y="-17.78" size="1.778" layer="95" xref="yes"/>
 </segment>
+<segment>
+<wire x1="167.64" y1="30.48" x2="162.56" y2="30.48" width="0.1524" layer="91"/>
+<label x="162.56" y="30.48" size="1.778" layer="95" rot="R180" xref="yes"/>
+<pinref part="SJ1" gate="G$1" pin="1"/>
+<wire x1="167.64" y1="30.48" x2="167.64" y2="27.94" width="0.1524" layer="91"/>
+</segment>
 </net>
 <net name="N$10" class="0">
@@
 </segment>
 </net>
+<net name="N$6" class="0">
+<segment>
+<pinref part="SJ1" gate="G$1" pin="2"/>
+<pinref part="SBUS" gate="A" pin="1"/>
+<wire x1="162.56" y1="22.86" x2="144.78" y2="22.86" width="0.1524" layer="91"/>
+</segment>
+</net>

Commit message: Moved SMA Connector
Connections:
- net GND: now also X1.GND1, X1.GND2, X1.GND3, X1.GND4
Changed lines of the file:
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@@
 <?xml version="1.0" encoding="utf-8"?>
 <!DOCTYPE eagle SYSTEM "eagle.dtd">
-<eagle version="8.6.0">
+<eagle version="9.0.0">
 <drawing>
 <settings>
@@
 <layers>
 <layer number="1" name="Top" color="4" fill="1" visible="no" active="no"/>
+<layer number="2" name="Route2" color="1" fill="3" visible="no" active="no"/>
+<layer number="3" name="Route3" color="4" fill="3" visible="no" active="no"/>
+<layer number="4" name="Route4" color="1" fill="4" visible="no" active="no"/>
+<layer number="5" name="Route5" color="4" fill="4" visible="no" active="no"/>
+<layer number="6" name="Route6" color="1" fill="8" visible="no" active="no"/>
+<layer number="7" name="Route7" color="4" fill="8" visible="no" active="no"/>
+<layer number="8" name="Route8" color="1" fill="2" visible="no" active="no"/>
+<layer number="9" name="Route9" color="4" fill="2" visible="no" active="no"/>
+<layer number="10" name="Route10" color="1" fill="7" visible="no" active="no"/>
+<layer number="11" name="Route11" color="4" fill="7" visible="no" active="no"/>
+<layer number="12" name="Route12" color="1" fill="5" visible="no" active="no"/>
+<layer number="13" name="Route13" color="4" fill="5" visible="no" active="no"/>
+<layer number="14" name="Route14" color="1" fill="6" visible="no" active="no"/>
+<layer number="15" name="Route15" color="4" fill="6" visible="no" active="no"/>
 <layer number="16" name="Bottom" color="1" fill="1" visible="no" active="no"/>
 <layer number="17" name="Pads" color="2" fill="1" visible="no" active="no"/>
@@
 <junction x="38.1" y="7.62"/>
 <pinref part="GND4" gate="1" pin="GND"/>
-</segment>
-<segment>
+<pinref part="X1" gate="G$1" pin="GND3"/>
+<pinref part="X1" gate="G$1" pin="GND4"/>
+<wire x1="48.26" y1="2.54" x2="53.34" y2="2.54" width="0.1524" layer="91"/>
+<wire x1="48.26" y1="2.54" x2="38.1" y2="2.54" width="0.1524" layer="91"/>
+<junction x="48.26" y="2.54"/>
+<junction x="38.1" y="2.54"/>
+<pinref part="X1" gate="G$1" pin="GND2"/>
+<pinref part="X1" gate="G$1" pin="GND1"/>
+<wire x1="53.34" y1="17.78" x2="48.26" y2="17.78" width="0.1524" layer="91"/>
+<wire x1="48.26" y1="17.78" x2="38.1" y2="17.78" width="0.1524" layer="91"/>
+<junction x="48.26" y="17.78"/>
+<wire x1="38.1" y1="17.78" x2="38.1" y2="12.7" width="0.1524" layer="91"/>
+<junction x="38.1" y="12.7"/>
+</segment>
+<segment>

Commit message: Changed some pins to simplify the layout
Connections:
- net !SS: now also U2.PB7(XTAL2/TOSC2/PCINT7); no longer U2.PC2(ADC2PCINT10)
- net STATUS: now also U2.PD0(RXD/PCINT16); no longer U2.PB7(XTAL2/TOSC2/PCINT7)
Changed lines of the file:
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@@
 </segment>
 <segment>
-<pinref part="U2" gate="G$1" pin="PC2(ADC2PCINT10)"/>
-<wire x1="129.54" y1="73.66" x2="134.62" y2="73.66" width="0.1524" layer="91"/>
-<label x="134.62" y="73.66" size="1.778" layer="95" xref="yes"/>
+<pinref part="U2" gate="G$1" pin="PB7(XTAL2/TOSC2/PCINT7)"/>
+<wire x1="129.54" y1="83.82" x2="134.62" y2="83.82" width="0.1524" layer="91"/>
+<label x="134.62" y="83.82" size="1.778" layer="95" xref="yes"/>
 </segment>
 </net>
@@
 <net name="STATUS" class="0">
 <segment>
-<pinref part="U2" gate="G$1" pin="PB7(XTAL2/TOSC2/PCINT7)"/>
-<wire x1="129.54" y1="83.82" x2="134.62" y2="83.82" width="0.1524" layer="91"/>
-<label x="134.62" y="83.82" size="1.778" layer="95" xref="yes"/>
-</segment>
-<segment>
 <pinref part="R6" gate="G$1" pin="2"/>
 <wire x1="55.88" y1="149.86" x2="55.88" y2="154.94" width="0.1524" layer="91"/>
 <label x="55.88" y="154.94" size="1.778" layer="95" rot="R90" xref="yes"/>
 </segment>
+<segment>
+<pinref part="U2" gate="G$1" pin="PD0(RXD/PCINT16)"/>
+<wire x1="129.54" y1="58.42" x2="137.16" y2="58.42" width="0.1524" layer="91"/>
+<label x="137.16" y="58.42" size="1.778" layer="95" xref="yes"/>
+</segment>
 </net>
